File: forty/40+/40+_pcb/40+_pcb.kicad_sch (KiCad schematic)
At the start: 1 part, among them U1 nRF52840

Commit message: firmware + qmk pcb start
Parts:
- added J1: USB_C_Receptacle_USB2.0_16P, symbol Connector:USB_C_Receptacle_USB2.0_16P
- added R1, R2: R, symbol Device:R
- added SW1: Switch, symbol ScottoKeebs:Placeholder_Switch
- added U2: USB6B1, Package_SO:SOIC-8_3.9x4.9mm_P1.27mm, symbol Power_Protection:USB6B1
- added U3: USBLC6-2SC6, Package_TO_SOT_SMD:SOT-23-6, symbol Power_Protection:USBLC6-2SC6
Connections:
- net D-: now reaches U1.AD4 (D-)
- net D-: now also J1.A7 (D-), J1.B7 (D-), U2.2 (I/O1), U2.7 (I/O1)
- net D+: now reaches U1.AD6 (D+)
- net D+: now also J1.A6 (D+), J1.B6 (D+), U2.3 (I/O2), U2.6 (I/O2)
- net GND: now reaches U1.B7 (VSS), U1.EP (VSS)
- net GND: now also U1.F23 (VSS_PA), J1.A1 (GND), J1.A12 (GND), J1.B1 (GND), J1.B12 (GND), R1.2, R2.2, U2.4 (GND), U2.5 (GND)
- new net: J1.A4 (VBUS), J1.A9 (VBUS), J1.B4 (VBUS), J1.B9 (VBUS)
- new net: J1.A5 (CC1), R1.1
- new net: J1.B5 (CC2), R2.1
- new net: U2.1 (VBUS), U2.8 (VBUS)
- no-connect marks 0 -> 3
Other:
- added sheet key-matrix (key-matrix.kicad_sch)
- moved on the sheet: U1

Commit message: macro w/ pcb start
Parts:
- added C1, C2, C3, C4, C5, C6, C7: C, symbol Device:C
- added D1: LED, symbol Device:LED
- added J2: Conn_01x02_Socket, symbol Connector:Conn_01x02_Socket
- added R3, R4, R5, R6, R7: R, symbol Device:R
- added U4: MCP73831-2-OT, Package_TO_SOT_SMD:SOT-23-5, symbol Battery_Management:MCP73831-2-OT
- SW1: footprint (none) -> Connector_JST:JST_EH_B2B-EH-A_1x02_P2.50mm_Vertical
- renumbered U2 to U1, U3 to U2, U1 to U3
Connections:
- net D+: now also R7.2; no longer U3.AD6 (D+)
- net D-: now also R6.2; no longer U3.AD4 (D-)
- net GND: now also SW1.1, U3.B5 (DEC4), U3.E24 (DEC6), U3.N24 (DEC5), C1.2, C2.1, C3.1, C4.1, C5.1, C6.2, C7.2, J2.2 (Pin_2), R4.1, U4.2 (V_{SS})
- net VBUS: now also J1.A4 (VBUS), J1.A9 (VBUS), J1.B4 (VBUS), J1.B9 (VBUS), U1.1 (VBUS), U1.8 (VBUS), U3.AD2 (VBUS), U3.Y2 (VDDH), C6.1, D1.2 (A), U4.4 (V_{DD})
- net at U3.A18 (DEC2): now also C3.2
- net VCC: now reaches U3.A22 (VDD), U3.AD14 (VDD), U3.AD23 (VDD), U3.B1 (VDD), U3.W1 (VDD)
- net VCC: now also C1.1, R5.1
- net at U3.AC13 (P0.18/~{RESET}): now also SW1.2, R5.2
- net at U3.AC5 (DECUSB): now also C5.2
- net at U3.C1 (DEC1): now also C2.2
- net at U3.D23 (DEC3): now also C4.2
- new net: R6.1, U3.AD4 (D-)
- new net: D1.1 (K), R3.2
- new net: R3.1, U4.1 (STAT)
- new net: C7.1, J2.1 (Pin_1), U4.3 (V_{BAT})
- new net: R4.2, U4.5 (PROG)
- new net: R7.1, U3.AD6 (D+)
Other:
- moved on the sheet: J1, R1, R2, SW1, U1, U2, U3
