File: macropad/pcb 4x4 macro/4x4_macro/4x4_macro.kicad_pcb (KiCad board)
At the start: 2 copper layers, 76.2 x 76.2 mm, 33 parts, among them U1 SuperMini nRF52840

Commit message: macro w/ pcb start
Routing:
- added copper zone on B.Cu, net (none)
- added copper zone on F.Cu, net (none)
Changed lines of the file:
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@@
-	)
-	(segment
-		(start 75.074 58.5808)
-		(end 75.311 58.3438)
-		(width 0.25)
-		(layer "B.Cu")
-		(net 22)
 	)
 	(segment
@@
 		(net 24)
 	)
+	(zone
+		(net 0)
+		(net_name "")
+		(layers "F.Cu" "B.Cu")
+		(hatch edge 0.5)
+		(connect_pads
+			(clearance 0.2)
+		)
+		(min_thickness 0.15)
+		(filled_areas_thickness no)
+		(fill yes
+			(thermal_gap 0.5)
+			(thermal_bridge_width 0.5)
+			(island_removal_mode 1)
+			(island_area_min 10)
+		)
+		(polygon
+			(pts
+				(xy 33.20415 21.77415) (xy 114.16665 21.77415) (xy 114.16665 102.73665) (xy 33.20415 102.73665)
+			)
+		)
+	)
 	(group ""
